File: VCO/VCO.sch (KiCad schematic (older format))
At the start: 17 parts

Commit message: VCO + DAC V2
Parts:
- removed U?: AD558JN, symbol AD558JN
- added AD1: AD5761R, symbol AD5761R
- added C4: 10nF, symbol C
- added J1: TEST, symbol TEST
- added VCC10, VCC16, VCC3, VCC5: VCC, symbol VCC
- gave numbers to parts that had none: 13
Connections:
- net labels added: STM_OUTPUT
- wire segments 34 -> 44

Commit message: Cleaned power supplies
Parts:
- removed VCC10, VCC16, VCC3, VCC5: VCC, symbol VCC
Connections:
- net labels added: VDD
- net labels removed: GNDD
- wire segments 44 -> 37
Other:
- note added: "VCC (analog supply) should be 16V\nVDD (digital supply) should be 3V or 3.3V"
Changed lines of the file:
@@
 	1    0    0    1
-$EndComp
-$Comp
-L VCC VCC5
-U 1 1 58C00244
-P 6950 1550
-F 0 "VCC5" H 6950 1400 50  0001 C CNN
-F 1 "VCC" H 6950 1700 50  0000 C CNB
-F 2 "" H 6950 1550 50  0000 C CNN
-F 3 "" H 6950 1550 50  0000 C CNN
-	1    6950 1550
-	1    0    0    -1
 $EndComp
 Text Notes 7400 7500 0    60   ~ 0
@@
 $EndComp
 $Comp
-L VCC #PWR07
-U 1 1 58C8271A
-P 7550 2000
-F 0 "#PWR07" H 7550 1850 50  0001 C CNN
-F 1 "VCC" H 7550 2150 50  0000 C CNN
-F 2 "" H 7550 2000 50  0000 C CNN
-F 3 "" H 7550 2000 50  0000 C CNN
-	1    7550 2000
-	0    -1   -1   0
-$EndComp
-$Comp
 L CONN_01X02 P?
 U 1 1 58C82797
@@
 $EndComp
 $Comp
-L VCC VCC10
-U 1 1 58C858D8
-P 5600 3100
-F 0 "VCC10" H 5600 2950 50  0001 C CNN
-F 1 "VCC" H 5600 3250 50  0000 C CNN
-F 2 "" H 5600 3100 50  0000 C CNN
-F 3 "" H 5600 3100 50  0000 C CNN
-	1    5600 3100
-	-1   0    0    1
-$EndComp
-$Comp
 L JACK_MONO J_Rec
 U 1 1 58D1CA56
@@
 $EndComp
 $Comp
-L GND #PWR?
-U 1 1 58DA8162
-P 3550 2700
-F 0 "#PWR?" H 3550 2450 50  0001 C CNN
-F 1 "GND" H 3550 2550 50  0000 C CNN
-F 2 "" H 3550 2700 50  0000 C CNN
-F 3 "" H 3550 2700 50  0000 C CNN
-	1    3550 2700
-	0    -1   -1   0
-$EndComp
-$Comp
-L GNDD #PWR?
-U 1 1 58DA91FA
-P 2500 3300
-F 0 "#PWR?" H 2500 3050 50  0001 C CNN
-F 1 "GNDD" H 2500 3150 50  0000 C CNN
-F 2 "" H 2500 3300 50  0000 C CNN
-F 3 "" H 2500 3300 50  0000 C CNN
-	1    2500 3300
-	0    1    1    0
-$EndComp
-$Comp
-L VCC VCC3
-U 1 1 58DAA9D9
-P 2250 3100
-F 0 "VCC3" H 2250 2950 50  0001 C CNN
-F 1 "VCC" H 2250 3250 50  0000 C CNN
-F 2 "" H 2250 3100 50  0000 C CNN
-F 3 "" H 2250 3100 50  0000 C CNN
-	1    2250 3100
-	0    -1   -1   0
-$EndComp
-$Comp
 L C C4
 U 1 1 58DABABF
@@
 	1    0    0    -1
 $EndComp
-$Comp
-L GND #PWR?
-U 1 1 58DACD57
+Text Label 2100 2700 2    60   ~ 0
+STM_OUTPUT
+Wire Wire Line
+	4800 2650 5400 2650
+Wire Wire Line
+	4800 2450 5400 2450
+Wire Wire Line
+	5150 2450 5150 3100
+Connection ~ 5150 2450
+Wire Wire Line
+	5150 3400 5150 3600
+Wire Wire Line
+	5150 4000 5150 4150
+Wire Wire Line
+	5250 2650 5250 2850
+Wire Wire Line
+	5250 2850 5400 2850
+Wire Wire Line
+	5400 2850 5400 2900
+Connection ~ 5250 2650
+Wire Wire Line
+	5400 3200 5400 3350
+Wire Wire Line
+	5300 2450 5300 1950
+Wire Wire Line
+	5300 1950 5550 1950
+Connection ~ 5300 2450
+Connection ~ 6250 2550
+Wire Wire Line
+	6950 3000 7350 3000
+Wire Wire Line
+	6950 2050 6950 3150
+Connection ~ 6950 2550
+Wire Wire Line
+	6950 2750 7050 2750
+Connection ~ 6950 2750
+Wire Wire Line
+	6950 1550 6950 1750
+Connection ~ 6950 3000
+Wire Wire Line
+	6950 3450 6950 3600
+Wire Wire Line
+	7900 3800 5450 3800
+Wire Wire Line
+	7900 2650 7900 3800
+Wire Wire Line
+	7650 3000 7900 3000
+Connection ~ 7900 3000
+Connection ~ 4500 2550
+Wire Wire Line
+	4300 2450 4300 2550
+Connection ~ 4300 2550
+Wire Wire Line
+	6600 2050 6600 2550
+Connection ~ 6600 2550
+Connection ~ 7900 2650
+Wire Wire Line
+	5750 1950 6250 1950
+Wire Wire Line
+	6250 1950 6250 2550
+Wire Wire Line
+	6000 2550 7050 2550
+Wire Wire Line
+	5600 2850 5600 3100
+Wire Wire Line
+	7650 2650 8400 2650
+Wire Wire Line
+	8400 2750 8400 2950
+Wire Wire Line
+	6700 2050 6700 2200
+Wire Wire Line
+	4500 2550 4250 2550
+Wire Wire Line
+	4250 2550 4250 2950
+Wire Wire Line
+	3500 2400 3800 2400
+Wire Wire Line
+	3800 2400 3800 2950
+Wire Wire Line
+	3800 2950 3850 2950
+Wire Wire Line
+	3500 2850 3700 2850
+Wire Wire Line
+	3700 2850 3700 2900
+Wire Wire Line
+	2100 2700 2500 2700
+Wire Wire Line
+	4500 2450 4500 2650
+$Comp
+L GND #PWR?
+U 1 1 58DA7165
+P 3500 2700
+F 0 "#PWR?" H 3500 2450 50  0001 C CNN
+F 1 "GND" H 3500 2550 50  0000 C CNN
+F 2 "" H 3500 2700 50  0000 C CNN
+F 3 "" H 3500 2700 50  0000 C CNN
+	1    3500 2700
+	0    -1   -1   0
+$EndComp
+$Comp
+L GND #PWR?
+U 1 1 58DA71BF
+P 2500 3300
+F 0 "#PWR?" H 2500 3050 50  0001 C CNN
+F 1 "GND" H 2500 3150 50  0000 C CNN
+F 2 "" H 2500 3300 50  0000 C CNN
+F 3 "" H 2500 3300 50  0000 C CNN
+	1    2500 3300
+	0    1    1    0
+$EndComp
+$Comp
+L VCC #PWR?
+U 1 1 58DA71F2
 P 3500 2250
-F 0 "#PWR?" H 3500 2000 50  0001 C CNN
-F 1 "GND" H 3500 2100 50  0000 C CNN
+F 0 "#PWR?" H 3500 2100 50  0001 C CNN
+F 1 "VCC" H 3500 2400 50  0000 C CNN
 F 2 "" H 3500 2250 50  0000 C CNN
 F 3 "" H 3500 2250 50  0000 C CNN
 	1    3500 2250
-	0    -1   -1   0
-$EndComp
-$Comp
-L VCC VCC16
-U 1 1 58DACD9B
-P 3550 2550
-F 0 "VCC16" H 3550 2400 50  0001 C CNN
-F 1 "VCC" H 3550 2700 50  0000 C CNN
-F 2 "" H 3550 2550 50  0000 C CNN
-F 3 "" H 3550 2550 50  0000 C CNN
-	1    3550 2550
 	0    1    1    0
 $EndComp
-Text Label 2100 2700 2    60   ~ 0
-STM_OUTPUT
-Wire Wire Line
-	4800 2650 5400 2650
-Wire Wire Line
-	4800 2450 5400 2450
-Wire Wire Line
-	5150 2450 5150 3100
-Connection ~ 5150 2450
-Wire Wire Line
-	5150 3400 5150 3600
-Wire Wire Line
-	5150 4000 5150 4150
-Wire Wire Line
-	5250 2650 5250 2850
-Wire Wire Line
-	5250 2850 5400 2850
-Wire Wire Line
-	5400 2850 5400 2900
-Connection ~ 5250 2650
-Wire Wire Line
-	5400 3200 5400 3350
-Wire Wire Line
-	5300 2450 5300 1950
-Wire Wire Line
-	5300 1950 5550 1950
-Connection ~ 5300 2450
-Connection ~ 6250 2550
-Wire Wire Line
-	6950 3000 7350 3000
-Wire Wire Line
-	6950 2050 6950 3150
-Connection ~ 6950 2550
-Wire Wire Line
-	6950 2750 7050 2750
-Connection ~ 6950 2750
-Wire Wire Line
-	6950 1550 6950 1750
-Connection ~ 6950 3000
-Wire Wire Line
-	6950 3450 6950 3600
-Wire Wire Line
-	7900 3800 5450 3800
-Wire Wire Line
-	7900 2650 7900 3800
-Wire Wire Line
-	7650 3000 7900 3000
-Connection ~ 7900 3000
-Wire Wire Line
-	4500 2450 4500 2650
-Connection ~ 4500 2550
-Wire Wire Line
-	4300 2450 4300 2550
-Connection ~ 4300 2550
-Wire Wire Line
-	6600 2050 6600 2550
-Connection ~ 6600 2550
-Connection ~ 7900 2650
-Wire Wire Line
-	5750 1950 6250 1950
-Wire Wire Line
-	6250 1950 6250 2550
-Wire Wire Line
-	6000 2550 7050 2550
-Wire Wire Line
-	5600 2850 5600 3100
-Wire Wire Line
-	7650 2650 8400 2650
-Wire Wire Line
-	8400 2750 8400 2950
-Wire Wire Line
-	6700 2050 6700 2200
-Wire Wire Line
-	4550 2600 4500 2600
-Wire Wire Line
-	4500 2600 4500 2550
-Wire Wire Line
-	4500 2550 4250 2550
-Wire Wire Line
-	4250 2550 4250 2950
-Wire Wire Line
-	3500 2400 3800 2400
-Wire Wire Line
-	3800 2400 3800 2950
-Wire Wire Line
-	3800 2950 3850 2950
-Wire Wire Line
-	3500 2700 3550 2700
-Wire Wire Line
-	2250 3100 2450 3100
-Wire Wire Line
-	2450 3100 2450 3150
-Wire Wire Line
-	2450 3150 2500 3150
-Wire Wire Line
-	3500 2850 3700 2850
-Wire Wire Line
-	3700 2850 3700 2900
-Wire Wire Line
-	3500 2550 3550 2550
-Wire Wire Line
-	2100 2700 2500 2700
+$Comp
+L VCC #PWR?
+U 1 1 58DA723D
+P 5600 3100
+F 0 "#PWR?" H 5600 2950 50  0001 C CNN
+F 1 "VCC" H 5600 3250 50  0000 C CNN
+F 2 "" H 5600 3100 50  0000 C CNN
+F 3 "" H 5600 3100 50  0000 C CNN
+	1    5600 3100
+	-1   0    0    1
+$EndComp
+$Comp
+L VDD #PWR?
+U 1 1 58DA7270
+P 2500 3150
+F 0 "#PWR?" H 2500 3000 50  0001 C CNN
+F 1 "VDD" H 2500 3300 50  0000 C CNN
+F 2 "" H 2500 3150 50  0000 C CNN
+F 3 "" H 2500 3150 50  0000 C CNN
+	1    2500 3150
+	0    -1   -1   0
+$EndComp
+Text Notes 1700 1800 0    60   ~ 0
+VCC (analog supply) should be 16V\nVDD (digital supply) should be 3V or 3.3V
+$Comp
+L GND #PWR?
+U 1 1 58DA7478
+P 3500 2550
+F 0 "#PWR?" H 3500 2300 50  0001 C CNN
+F 1 "GND" H 3500 2400 50  0000 C CNN
+F 2 "" H 3500 2550 50  0000 C CNN
+F 3 "" H 3500 2550 50  0000 C CNN
+	1    3500 2550
+	0    -1   -1   0
+$EndComp
+$Comp
+L VCC #PWR?
+U 1 1 58DA7621
+P 7550 2000
+F 0 "#PWR?" H 7550 1850 50  0001 C CNN
+F 1 "VCC" H 7550 2150 50  0000 C CNN
+F 2 "" H 7550 2000 50  0000 C CNN
+F 3 "" H 7550 2000 50  0000 C CNN
+	1    7550 2000
+	0    -1   -1   0
+$EndComp
+$Comp
+L VCC #PWR?
+U 1 1 58DA7679
+P 6950 1550
+F 0 "#PWR?" H 6950 1400 50  0001 C CNN
+F 1 "VCC" H 6950 1700 50  0000 C CNN
+F 2 "" H 6950 1550 50  0000 C CNN
+F 3 "" H 6950 1550 50  0000 C CNN
+	1    6950 1550
+	1    0    0    -1
+$EndComp
 $EndSCHEMATC

Commit message: VCO maJ
Parts:
- removed P?: CONN_01X02, symbol CONN_01X02
- added C5, C6: 100nF, symbol C
- added H1: HEADER_ALIM, symbol CONN_01X03
- added H2: HEADER_DAC, symbol CONN_01X07
- C4: value 10nF -> 100nF
- renumbered J_Rec to J_Rec1, J_Tri to J_Tri1
Connections:
- net labels added: SCLK, SDO, ~ALERT, ~CLEAR, ~LDAC, ~RESET, ~SYNC
- net labels removed: STM_OUTPUT
- wire segments 37 -> 39
- no-connect marks 0 -> 1
Other:
- note added: "Output de la STM32"
- moved on the sheet: C4
Changed lines of the file:
@@
 $EndComp
 $Comp
-L GND #PWR01
+L GND #PWR8
 U 1 1 58BED608
 P 5150 4150
-F 0 "#PWR01" H 5150 3900 50  0001 C CNN
+F 0 "#PWR8" H 5150 3900 50  0001 C CNN
 F 1 "GND" H 5150 4000 50  0000 C CNN
 F 2 "" H 5150 4150 50  0000 C CNN
@@
 $EndComp
 $Comp
-L GND #PWR02
+L GND #PWR9
 U 1 1 58BEDD61
 P 5400 3350
-F 0 "#PWR02" H 5400 3100 50  0001 C CNN
+F 0 "#PWR9" H 5400 3100 50  0001 C CNN
 F 1 "GND" H 5400 3200 50  0000 C CNN
 F 2 "" H 5400 3350 50  0000 C CNN
@@
 $EndComp
 $Comp
-L GND #PWR03
+L GND #PWR15
 U 1 1 58BF02DC
 P 6950 3600
-F 0 "#PWR03" H 6950 3350 50  0001 C CNN
+F 0 "#PWR15" H 6950 3350 50  0001 C CNN
 F 1 "GND" H 6950 3450 50  0000 C CNN
 F 2 "" H 6950 3600 50  0000 C CNN
@@
 $EndComp
 $Comp
-L GND #PWR04
+L GND #PWR7
 U 1 1 58BEEBFA
 P 4300 2150
-F 0 "#PWR04" H 4300 1900 50  0001 C CNN
+F 0 "#PWR7" H 4300 1900 50  0001 C CNN
 F 1 "GND" H 4300 2000 50  0000 C CNN
 F 2 "" H 4300 2150 50  0000 C CNN
@@
 $EndComp
 $Comp
-L GND #PWR06
+L GND #PWR10
 U 1 1 58C825A1
 P 5600 2250
-F 0 "#PWR06" H 5600 2000 50  0001 C CNN
+F 0 "#PWR10" H 5600 2000 50  0001 C CNN
 F 1 "GND" H 5600 2100 50  0000 C CNN
 F 2 "" H 5600 2250 50  0000 C CNN
@@
 $EndComp
 $Comp
-L CONN_01X02 P?
-U 1 1 58C82797
-P 7750 2050
-F 0 "P?" H 7750 2200 50  0000 C CNN
-F 1 "CONN_01X02" V 7850 2050 50  0000 C CNN
-F 2 "" H 7750 2050 50  0000 C CNN
-F 3 "" H 7750 2050 50  0000 C CNN
-	1    7750 2050
-	1    0    0    -1
-$EndComp
-$Comp
-L GND #PWR08
+L GND #PWR18
 U 1 1 58C8525C
-P 7550 2100
-F 0 "#PWR08" H 7550 1850 50  0001 C CNN
-F 1 "GND" H 7550 1950 50  0000 C CNN
-F 2 "" H 7550 2100 50  0000 C CNN
-F 3 "" H 7550 2100 50  0000 C CNN
-	1    7550 2100
+P 4650 3450
+F 0 "#PWR18" H 4650 3200 50  0001 C CNN
+F 1 "GND" H 4650 3300 50  0000 C CNN
+F 2 "" H 4650 3450 50  0000 C CNN
+F 3 "" H 4650 3450 50  0000 C CNN
+	1    4650 3450
 	0    1    1    0
 $EndComp
@@
 $EndComp
 $Comp
-L GND #PWR09
+L GND #PWR12
 U 1 1 58C856DC
 P 5900 3100
-F 0 "#PWR09" H 5900 2850 50  0001 C CNN
+F 0 "#PWR12" H 5900 2850 50  0001 C CNN
 F 1 "GND" H 5900 2950 50  0000 C CNN
 F 2 "" H 5900 3100 50  0000 C CNN
@@
 $EndComp
 $Comp
-L JACK_MONO J_Rec
+L JACK_MONO J_Rec1
 U 1 1 58D1CA56
 P 8700 2650
-F 0 "J_Rec" H 8700 2900 60  0000 C CNN
-F 1 "JACK_MONO" H 8950 2700 60  0000 C CNN
+F 0 "J_Rec1" H 8700 2900 60  0000 C CNN
+F 1 "JACK_MONO" H 9150 2800 60  0000 C CNN
 F 2 "" H 8950 2700 60  0000 C CNN
 F 3 "" H 8950 2700 60  0000 C CNN
@@
 $EndComp
 $Comp
-L GND #PWR?
+L GND #PWR19
 U 1 1 58D1CBD1
 P 8400 2950
-F 0 "#PWR?" H 8400 2700 50  0001 C CNN
+F 0 "#PWR19" H 8400 2700 50  0001 C CNN
 F 1 "GND" H 8400 2800 50  0000 C CNN
 F 2 "" H 8400 2950 50  0000 C CNN
@@
 $EndComp
 $Comp
-L JACK_MONO J_Tri
+L JACK_MONO J_Tri1
 U 1 1 58D1D643
 P 6600 1750
-F 0 "J_Tri" V 6650 2100 60  0000 C CNN
+F 0 "J_Tri1" V 6650 2100 60  0000 C CNN
 F 1 "JACK_MONO" V 6900 1800 60  0000 C CNN
 F 2 "" H 6850 1800 60  0000 C CNN
@@
 $EndComp
 $Comp
-L GND #PWR?
+L GND #PWR13
 U 1 1 58D1DBA4
 P 6700 2200
-F 0 "#PWR?" H 6700 1950 50  0001 C CNN
+F 0 "#PWR13" H 6700 1950 50  0001 C CNN
 F 1 "GND" H 6700 2050 50  0000 C CNN
 F 2 "" H 6700 2200 50  0000 C CNN
@@
 L C C4
 U 1 1 58DABABF
-P 3700 3050
-F 0 "C4" H 3725 3150 50  0000 L CNN
-F 1 "10nF" H 3725 2950 50  0000 L CNN
-F 2 "" H 3738 2900 50  0000 C CNN
-F 3 "" H 3700 3050 50  0000 C CNN
-	1    3700 3050
-	1    0    0    -1
-$EndComp
-$Comp
-L GND #PWR?
+P 3850 3250
+F 0 "C4" H 3875 3350 50  0000 L CNN
+F 1 "100nF" H 3875 3150 50  0000 L CNN
+F 2 "" H 3888 3100 50  0000 C CNN
+F 3 "" H 3850 3250 50  0000 C CNN
+	1    3850 3250
+	1    0    0    -1
+$EndComp
+$Comp
+L GND #PWR5
 U 1 1 58DABBD6
-P 3700 3200
-F 0 "#PWR?" H 3700 2950 50  0001 C CNN
-F 1 "GND" H 3700 3050 50  0000 C CNN
-F 2 "" H 3700 3200 50  0000 C CNN
-F 3 "" H 3700 3200 50  0000 C CNN
-	1    3700 3200
-	1    0    0    -1
-$EndComp
-Text Label 2100 2700 2    60   ~ 0
-STM_OUTPUT
+P 3850 3400
+F 0 "#PWR5" H 3850 3150 50  0001 C CNN
+F 1 "GND" H 3850 3250 50  0000 C CNN
+F 2 "" H 3850 3400 50  0000 C CNN
+F 3 "" H 3850 3400 50  0000 C CNN
+	1    3850 3400
+	1    0    0    -1
+$EndComp
 Wire Wire Line
 	4800 2650 5400 2650
@@
 	3500 2850 3700 2850
 Wire Wire Line
-	3700 2850 3700 2900
+	3700 2850 3700 3100
 Wire Wire Line
 	2100 2700 2500 2700
@@
 	4500 2450 4500 2650
 $Comp
-L GND #PWR?
+L GND #PWR4
 U 1 1 58DA7165
 P 3500 2700
-F 0 "#PWR?" H 3500 2450 50  0001 C CNN
+F 0 "#PWR4" H 3500 2450 50  0001 C CNN
 F 1 "GND" H 3500 2550 50  0000 C CNN
 F 2 "" H 3500 2700 50  0000 C CNN
@@
 $EndComp
 $Comp
-L GND #PWR?
+L GND #PWR2
 U 1 1 58DA71BF
 P 2500 3300
-F 0 "#PWR?" H 2500 3050 50  0001 C CNN
+F 0 "#PWR2" H 2500 3050 50  0001 C CNN
 F 1 "GND" H 2500 3150 50  0000 C CNN
 F 2 "" H 2500 3300 50  0000 C CNN
@@
 $EndComp
 $Comp
-L VCC #PWR?
+L VCC #PWR6
 U 1 1 58DA71F2
-P 3500 2250
-F 0 "#PWR?" H 3500 2100 50  0001 C CNN
-F 1 "VCC" H 3500 2400 50  0000 C CNN
-F 2 "" H 3500 2250 50  0000 C CNN
-F 3 "" H 3500 2250 50  0000 C CNN
-	1    3500 2250
+P 3800 2250
+F 0 "#PWR6" H 3800 2100 50  0001 C CNN
+F 1 "VCC" H 3800 2400 50  0000 C CNN
+F 2 "" H 3800 2250 50  0000 C CNN
+F 3 "" H 3800 2250 50  0000 C CNN
+	1    3800 2250
 	0    1    1    0
 $EndComp
 $Comp
-L VCC #PWR?
+L VCC #PWR11
 U 1 1 58DA723D
 P 5600 3100
-F 0 "#PWR?" H 5600 2950 50  0001 C CNN
+F 0 "#PWR11" H 5600 2950 50  0001 C CNN
 F 1 "VCC" H 5600 3250 50  0000 C CNN
 F 2 "" H 5600 3100 50  0000 C CNN
@@
 $EndComp
 $Comp
-L VDD #PWR?
+L VDD #PWR1
 U 1 1 58DA7270
 P 2500 3150
-F 0 "#PWR?" H 2500 3000 50  0001 C CNN
+F 0 "#PWR1" H 2500 3000 50  0001 C CNN
 F 1 "VDD" H 2500 3300 50  0000 C CNN
 F 2 "" H 2500 3150 50  0000 C CNN
@@
 	0    -1   -1   0
 $EndComp
-Text Notes 1700 1800 0    60   ~ 0
+Text Notes 1650 1800 0    60   ~ 0
 VCC (analog supply) should be 16V\nVDD (digital supply) should be 3V or 3.3V
 $Comp
-L GND #PWR?
+L GND #PWR3
 U 1 1 58DA7478
 P 3500 2550
-F 0 "#PWR?" H 3500 2300 50  0001 C CNN
+F 0 "#PWR3" H 3500 2300 50  0001 C CNN
 F 1 "GND" H 3500 2400 50  0000 C CNN
 F 2 "" H 3500 2550 50  0000 C CNN
@@
 $EndComp
 $Comp
-L VCC #PWR?
+L VCC #PWR16
 U 1 1 58DA7621
-P 7550 2000
-F 0 "#PWR?" H 7550 1850 50  0001 C CNN
-F 1 "VCC" H 7550 2150 50  0000 C CNN
-F 2 "" H 7550 2000 50  0000 C CNN
-F 3 "" H 7550 2000 50  0000 C CNN
-	1    7550 2000
-	0    -1   -1   0
-$EndComp
-$Comp
-L VCC #PWR?
+P 4650 3250
+F 0 "#PWR16" H 4650 3100 50  0001 C CNN
+F 1 "VCC" H 4650 3400 50  0000 C CNN
+F 2 "" H 4650 3250 50  0000 C CNN
+F 3 "" H 4650 3250 50  0000 C CNN
+	1    4650 3250
+	0    -1   -1   0
+$EndComp
+$Comp
+L VCC #PWR14
 U 1 1 58DA7679
 P 6950 1550
-F 0 "#PWR?" H 6950 1400 50  0001 C CNN
+F 0 "#PWR14" H 6950 1400 50  0001 C CNN
 F 1 "VCC" H 6950 1700 50  0000 C CNN
 F 2 "" H 6950 1550 50  0000 C CNN
@@
 	1    0    0    -1
 $EndComp
+$Comp
+L CONN_01X03 H1
+U 1 1 58E394FA
+P 4850 3350
+F 0 "H1" H 4850 3550 50  0000 C CNN
+F 1 "HEADER_ALIM" V 4950 3350 50  0000 C CNN
+F 2 "" H 4850 3350 50  0000 C CNN
+F 3 "" H 4850 3350 50  0000 C CNN
+	1    4850 3350
+	1    0    0    -1
+$EndComp
+$Comp
+L VDD #PWR17
+U 1 1 58E3978D
+P 4650 3350
+F 0 "#PWR17" H 4650 3200 50  0001 C CNN
+F 1 "VDD" H 4650 3500 50  0000 C CNN
+F 2 "" H 4650 3350 50  0000 C CNN
+F 3 "" H 4650 3350 50  0000 C CNN
+	1    4650 3350
+	0    -1   -1   0
+$EndComp
+Wire Wire Line
+	3500 2250 3800 2250
+NoConn ~ 2500 2250
+Text Label 2500 2400 2    60   ~ 0
+SDO
+Text Label 3900 1600 3    60   ~ 0
+SDO
+Text Label 2500 2550 2    60   ~ 0
+~LDAC
+Text Label 4000 1600 3    60   ~ 0
+~LDAC
+$Comp
+L C C6
+U 1 1 58E3F33A
+P 2050 3250
+F 0 "C6" H 2075 3350 50  0000 L CNN
+F 1 "100nF" H 2075 3150 50  0000 L CNN
+F 2 "" H 2088 3100 50  0000 C CNN
+F 3 "" H 2050 3250 50  0000 C CNN
+	1    2050 3250
+	1    0    0    -1
+$EndComp
+$Comp
+L CONN_01X07 H2
+U 1 1 58E42010
+P 4200 1400
+F 0 "H2" H 4200 1800 50  0000 C CNN
+F 1 "HEADER_DAC" V 4300 1400 50  0000 C CNN
+F 2 "" H 4200 1400 50  0000 C CNN
+F 3 "" H 4200 1400 50  0000 C CNN
+	1    4200 1400
+	0    -1   -1   0
+$EndComp
+Text Label 2500 2850 2    60   ~ 0
+~SYNC
+Text Label 4100 1600 3    60   ~ 0
+~SYNC
+Text Label 2500 3000 2    60   ~ 0
+SCLK
+Text Label 4200 1600 3    60   ~ 0
+SCLK
+Wire Wire Line
+	3700 3100 3850 3100
+Text Label 3500 3000 0    60   ~ 0
+~RESET
+Text Label 4300 1600 3    60   ~ 0
+~RESET
+Text Label 3500 3150 0    60   ~ 0
+~CLEAR
+Text Label 4400 1600 3    60   ~ 0
+~CLEAR
+Text Label 3500 3300 0    60   ~ 0
+~ALERT
+Text Label 4500 1600 3    60   ~ 0
+~ALERT
+Text Notes 1150 2750 0    60   ~ 0
+Output de la STM32
+$Comp
+L C C5
+U 1 1 58E45976
+P 3600 2050
+F 0 "C5" H 3625 2150 50  0000 L CNN
+F 1 "100nF" H 3625 1950 50  0000 L CNN
+F 2 "" H 3638 1900 50  0000 C CNN
+F 3 "" H 3600 2050 50  0000 C CNN
+	1    3600 2050
+	1    0    0    -1
+$EndComp

Commit message: VCO avec empreintes
Parts:
- removed H2: HEADER_DAC, symbol CONN_01X07
- removed J_Tri1: JACK_MONO, symbol JACK_MONO
- removed U1, U2: TL081, symbol TL081
- added H2: HEADER_DAC, Pin_Headers:Pin_Header_Straight_1x08_Pitch2.54mm, symbol CONN_01X08
- added SW1: SWITCH_INV, switch:switch, symbol SWITCH_INV
- added U1: LM324, Housings_DIP:DIP-14_W7.62mm, symbol LM324
- AD1: footprint (none) -> Housings_SSOP:TSSOP-16_4.4x5mm_Pitch0.65mm
- C1, C2, C3, C4, C5, C6: footprint (none) -> Capacitors_ThroughHole:C_Axial_L5.1mm_D3.1mm_P7.50mm_Horizontal
- H1: footprint (none) -> bornier:Bornier_3pins
- I1: renamed from J1; footprint (none) -> test:test
- J1: renamed from J_Rec1; value JACK_MONO -> JACK_STEREO; footprint (none) -> jack:jack-stereo
- Q1: footprint (none) -> TO_SOT_Packages_THT:TO-92_Inline_Wide
- R1, R2, R3, R4, R5, R6, R7: footprint (none) -> Resistors_ThroughHole:R_Axial_DIN0207_L6.3mm_D2.5mm_P7.62mm_Horizontal
Connections:
- net labels added: SDI
- wire segments 39 -> 50
Other:
- note removed: "Output de la STM32"
- moved on the sheet: C5, J1
